File: FeriNixie ZM1177 Clock.kicad_pcb (KiCad board)
At the start: 4 copper layers, 153.5 x 49 mm, 256 parts, among them Q1 C20069138, Q10 C20069138, Q11 C20069138, Q12 C20069138, Q13 C20069138, Q14 C20069138, Q15 C20069138, Q16 C20069138, Q17 C20069138, Q18 C20069138, Q19 C20069138, Q2 C20069138, Q20 C20069138, Q21 C20069138, Q22 C20069138, Q23 C20069138, Q24 C20069138, Q25 C20069138, Q26 C20069138, Q27 C20069138, Q28 C20069138, Q29 C20069138, Q3 C20069138, Q30 C20069138, Q31 C20069138, Q32 C20069138, Q33 C20069138, Q34 C20069138, Q35 C20069138, Q36 C20069138, Q37 C20069138, Q38 C20069138, Q39 C20069138, Q4 C20069138, Q40 C20069138, Q41 C20069138, Q42 C20069138, Q43 C20069138, Q44 C20069138, Q45 C20069138, Q46 C20069138, Q47 C20069138, Q48 C20069138, Q49 C20069138, Q5 C20069138, Q50 C20069138, Q51 C20069138, Q52 C20069138, Q53 C20069138, Q54 C20069138, Q55 C20069138, Q56 C20069138, Q57 C20069138, Q58 C20069138, Q59 C20069138, Q6 C20069138, Q60 C20069138, Q61 C20069138, Q62 C20069138, Q63 C20069138, Q64 C20069138, Q65 C20069138, Q66 C20069138, Q67 C20069138, Q68 C20069138, Q69 C20069138, Q7 C20069138, Q70 C20069138, Q8 C20069138, Q9 C20069138, U1 74HC595D,118, U2 74HC595D,118, U3 74HC595D,118, U4 74HC595D,118, U5 74HC595D,118, U6 74HC595D,118, U7 74HC595D,118, U8 74HC595D,118, U9 74HC595D,118

Commit message: Significant upgrades
Parts:
- added ?: , , F.Cu at (43.0, 35.7)
- added ?: , , F.Cu at (43.0, 32.7)
- moved R87 50.3 mm to (128.0, 38.2), turned to 180 degrees
- moved R82 36.1 mm to (109.6, 62.2), turned to 180 degrees
- moved R81 34.3 mm to (106.0, 62.2), turned to 180 degrees
- moved R80 33.2 mm to (104.2, 61.7), turned to 90 degrees
- moved R79 31.4 mm to (103.2, 61.7), turned to 90 degrees
- moved R76 22.1 mm to (102.3, 39.6), turned to 0 degrees
- moved R86 22.1 mm to (113.2, 62.2), turned to 180 degrees
- moved R85 21.1 mm to (118.2, 61.8), turned to 90 degrees
- moved R84 19.0 mm to (117.2, 61.8), turned to 90 degrees
- moved R83 16.8 mm to (116.2, 61.8), turned to 90 degrees
- moved R77 1.20 mm to (101.2, 61.7)
- moved R78 1.20 mm to (102.2, 61.7)
- moved R72 0.20 mm to (98.2, 61.7)
- moved R73 0.20 mm to (99.2, 61.7)
- moved R74 0.20 mm to (100.2, 61.7)
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Routing:
- net GND: track 31.8 -> 67.6 mm, vias 29 -> 40
- net Net-(U5-Q1): track 9.72 -> 32.0 mm, vias 0 -> 2
- net Net-(Q38-B): track 23.5 -> 1.71 mm, vias 2 -> 0
- net Net-(Q40-B): track 0.49 -> 19.3 mm, vias 1 -> 2
- net Net-(Q47-B): track 0.00 -> 18.2 mm, vias 0 -> 2
- net Net-(Q39-B): track 0.49 -> 17.9 mm, vias 1 -> 2
- net Net-(Q46-B): track 0.00 -> 14.5 mm, vias 0 -> 2
- net Net-(Q41-B): track 0.00 -> 11.6 mm, vias 0 -> 2
- net Net-(U5-Q7): track 0.00 -> 11.4 mm, vias 0 -> 2
- net Net-(Q45-B): track 0.00 -> 10.7 mm, vias 0 -> 2
- net Net-(U6-Q1): track 0.00 -> 10.4 mm, vias 0 -> 2
- net Net-(U6-Q2): track 0.00 -> 10.3 mm, vias 0 -> 2
- net Net-(U5-Q5): track 0.00 -> 8.54 mm
- net Net-(U5-Q6): track 0.00 -> 8.51 mm
- net Net-(U5-Q4): track 0.00 -> 8.45 mm
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- added copper zone on B.Cu, net GND
- added copper zone on F.Cu, net GND
- added copper zone on In1.Cu, net GND
- added copper zone on In2.Cu, net GND

Commit message: publish updates
Parts:
- added BT1: Battery_Cell, Battery:BatteryHolder_Keystone_1042_1x18650, F.Cu at (239.2, 72.1)
- added C18: C, Capacitor_THT:C_Radial_D8.0mm_H11.5mm_P3.50mm, F.Cu at (266.7, 110.7)
- added C32: CL31A226KAHNNNE, Capacitor_SMD:C_1206_3216Metric, F.Cu at (266.5, 85.1)
- added C33: CL31A226KAHNNNE, Capacitor_SMD:C_1206_3216Metric, F.Cu at (266.5, 88.5)
- added C34: CL10A106KP8NNNC, Capacitor_SMD:C_0603_1608Metric, F.Cu at (261.7, 84.7)
- added C35: CL10A106KP8NNNC, Capacitor_SMD:C_0603_1608Metric, F.Cu at (261.7, 87.2)
- added C36: CL10A106KP8NNNC, Capacitor_SMD:C_0603_1608Metric, F.Cu at (261.7, 89.7)
- added C37: CL31A226KAHNNNE, Capacitor_SMD:C_1206_3216Metric, F.Cu at (266.5, 91.8)
- added C38: CL31A226KAHNNNE, Capacitor_SMD:C_1206_3216Metric, F.Cu at (266.5, 95.2)
- added C39: CL10A106KP8NNNC, Capacitor_SMD:C_0603_1608Metric, F.Cu at (261.7, 92.2)
- added L1: FTM201610C1R0MCTA, JLCPCB_Imported:L0806, F.Cu at (277.2, 102.7)
- added R137: R, Resistor_THT:R_Axial_DIN0414_L11.9mm_D4.5mm_P15.24mm_Horizontal, F.Cu at (220.3, 102.7)
- added R138: 0603WAF200KT5E, Resistor_SMD:R_0603_1608Metric, F.Cu at (261.7, 94.8)
- added R139: 0603WAF200KT5E, Resistor_SMD:R_0603_1608Metric, F.Cu at (261.7, 97.3)
- added R254: 5.1K, Resistor_SMD:R_0402_1005Metric, F.Cu at (281.7, 107.0)
- added R255: 5.1K, Resistor_SMD:R_0402_1005Metric, F.Cu at (281.7, 108.9)
- added R256: 10K, Resistor_SMD:R_0402_1005Metric, F.Cu at (281.7, 110.9)
- added REF**: MountingHole_4.3mm_M4, MountingHole:MountingHole_4.3mm_M4, F.Cu at (102.2, 80.0)
- added REF**: MountingHole_4.3mm_M4, MountingHole:MountingHole_4.3mm_M4, F.Cu at (174.0, 99.5)
- added REF**: MountingHole_2.2mm_M2, MountingHole:MountingHole_2.2mm_M2, F.Cu at (154.5, 78.0)
- added REF**: MountingHole_2.2mm_M2, MountingHole:MountingHole_2.2mm_M2, F.Cu at (50.0, 28.5)
- added REF**: MountingHole_2.2mm_M2, MountingHole:MountingHole_2.2mm_M2, F.Cu at (154.5, 28.5)
- added REF**: MountingHole_4.3mm_M4, MountingHole:MountingHole_4.3mm_M4, F.Cu at (30.5, 99.5)
- added REF**: MountingHole_4.3mm_M4, MountingHole:MountingHole_4.3mm_M4, F.Cu at (102.2, 30.5)
- added REF**: MountingHole_2.2mm_M2, MountingHole:MountingHole_2.2mm_M2, F.Cu at (50.0, 78.0)
- added REF**: MountingHole_4.3mm_M4, MountingHole:MountingHole_4.3mm_M4, F.Cu at (174.0, 50.0)
- added REF**: MountingHole_4.3mm_M4, MountingHole:MountingHole_4.3mm_M4, F.Cu at (30.5, 50.0)
- added U10: RP2040-Tiny, NixFootprints:RP2040-Tiny Package Extra Clearance, F.Cu at (209.3, 95.0)
- added U11: NCH8200HV, NixFootprints:NCH8200HV Through-Hole, F.Cu at (250.1, 92.5)
- added U12: 1SMA4740A_C19077479, JLCPCB_Imported:SMA_L4.3-W2.6-LS5.0-RD, F.Cu at (278.6, 98.9)
- added U13: IP5306, JLCPCB_Imported:ESOP-8_L4.9-W3.9-P1.27-LS6.0-BL-EP, F.Cu at (277.0, 110.0)
- added U14: TYPE-C_16PIN_2MD(073), JLCPCB_Imported:USB-C-SMD_TYPE-C-16PIN-2MD-073, F.Cu at (269.2, 100.4)
- added U15: KT-0603R, JLCPCB_Imported:LED-SMD_L1.6-W0.8-R-RD, F.Cu at (277.7, 84.8)
- added U16: KT-0603R, JLCPCB_Imported:LED-SMD_L1.6-W0.8-R-RD, F.Cu at (277.7, 87.4)
- added U17: KT-0603R, JLCPCB_Imported:LED-SMD_L1.6-W0.8-R-RD, F.Cu at (277.7, 90.1)
- added U18: KT-0603R, JLCPCB_Imported:LED-SMD_L1.6-W0.8-R-RD, F.Cu at (277.7, 92.8)
- added U19: TS-1187A-B-A-B, JLCPCB_Imported:SW-SMD_4P-L5.1-W5.1-P3.70-LS6.5-TL_H1.5, F.Cu at (195.1, 42.7)
- C1, C2, C3, C4, C5, C6: footprint Capacitor_SMD:C_1206_3216Metric -> Resistor_SMD:R_1206_3216Metric
- moved R100 82.1 mm to (117.5, 8.19)
- moved R101 82.1 mm to (117.5, 10.2)
- moved R102 82.1 mm to (117.5, 12.2)
- moved R103 82.1 mm to (117.5, 14.2)
- moved R104 82.1 mm to (117.5, 16.1)
- moved R105 82.1 mm to (120.4, -3.75)
- moved R106 82.1 mm to (120.4, -1.76)
- moved R108 82.1 mm to (120.4, 2.22)
- moved R109 82.1 mm to (120.4, 4.21)
- moved R110 82.1 mm to (120.4, 6.20)
- moved R111 82.1 mm to (120.4, 8.19)
- moved R112 82.1 mm to (120.4, 10.2)
- moved R113 82.1 mm to (120.4, 12.2)
- moved R114 82.1 mm to (120.4, 14.2)
- moved R115 82.1 mm to (120.4, 16.1)
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Other:
- board size 153.5 x 49 mm -> 153.5 x 98.5 mm

Commit message: Update FeriNixie ZM1177 Clock.kicad_pcb
Parts:
- removed R256: 10K, Resistor_SMD:R_0402_1005Metric
- removed U19: TS-1187A-B-A-B, JLCPCB_Imported:SW-SMD_4P-L5.1-W5.1-P3.70-LS6.5-TL_H1.5
- added ?: , , F.Cu at (45.2, 80.2)
- added ?: , , F.Cu at (45.2, 83.2)
- added REF**: BarrelJack_CUI_PJ-063AH_Horizontal, Connector_BarrelJack:BarrelJack_CUI_PJ-063AH_Horizontal, F.Cu at (41.8, 91.2)
- moved U12 217.8 mm to (60.8, 98.9)
- moved C18 217.4 mm to (51.0, 83.2), turned to -90 degrees
- moved U15 208.0 mm to (72.2, 116.8), turned to 90 degrees
- moved C33 206.7 mm to (60.5, 105.1), turned to 90 degrees
- moved L1 206.0 mm to (71.2, 101.9)
- moved U16 205.8 mm to (74.0, 116.8), turned to -90 degrees
- moved U13 205.5 mm to (71.5, 109.2)
- moved R254 205.0 mm to (77.9, 84.5), turned to 90 degrees
- moved C39 203.8 mm to (57.9, 95.6), turned to 180 degrees
- moved U17 203.7 mm to (75.8, 116.8), turned to 90 degrees
- moved C37 203.1 mm to (63.9, 105.1), turned to 90 degrees
- moved R255 202.7 mm to (80.4, 84.5), turned to 90 degrees
- moved U18 201.6 mm to (77.6, 116.8), turned to -90 degrees
- moved C38 199.5 mm to (67.2, 105.1), turned to 90 degrees
- moved C34 198.4 mm to (65.6, 115.1)
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Routing:
- net GND: track 67.6 -> 188.2 mm, vias 40 -> 41
- net USB5V: track 0.00 -> 52.9 mm, vias 0 -> 2
- net +5V: track 16.9 -> 68.4 mm
- net VBAT: track 0.00 -> 21.5 mm
- net Net-(U13-VIN): track 0.00 -> 18.7 mm, vias 0 -> 1
- net Net-(U13-LED3): track 0.00 -> 16.9 mm
- net +170V: track 138.2 -> 153.3 mm
- net Net-(U13-LED2): track 0.00 -> 8.73 mm
- net Net-(U13-LED1): track 0.00 -> 6.24 mm
- net Net-(U13-SW): track 0.00 -> 4.72 mm
- net Net-(U14-CC2): track 0.00 -> 1.69 mm
- net Net-(U14-CC1): track 0.00 -> 1.50 mm
- net Net-(C36-Pad2): track 0.00 -> 1.50 mm
- net Net-(C34-Pad2): track 0.00 -> 1.50 mm

Commit message: PCB updates
Other:
- board text added: "25 50 75 100"
Changed lines of the file:
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@@
 			(at 0.036081 6.974981 0)
 			(layer "F.Fab")
+			(hide yes)
 			(effects
 				(font
@@
 		(layer "Edge.Cuts")
 	)
+	(gr_text "25 50 75 100"
+		(at 75.1 119.2 0)
+		(layer "F.SilkS")
+		(effects
+			(font
+				(size 1 0.8)
+				(thickness 0.2)
+				(bold yes)
+			)
+			(justify top)
+		)
+	)
 	(segment

Commit message: Lots of improvements and adjustments
Parts:
- added R140: 100K, Resistor_SMD:R_1206_3216Metric, F.Cu at (62.0, 101.6)
- added REF**: PinHeader_1x06_P2.54mm_Vertical, Connector_PinHeader_2.54mm:PinHeader_1x06_P2.54mm_Vertical, F.Cu at (49.5, 117.0)
- added REF**: PinHeader_1x06_P2.54mm_Vertical, Connector_PinHeader_2.54mm:PinHeader_1x06_P2.54mm_Vertical, F.Cu at (30.5, 57.5)
- added SW: , NixFootprints:SW_SPST_R1966ABLKBLKFR, F.Cu at (102.2, 110.0)
- C1, C2, C3, C4, C5, C6: footprint Resistor_SMD:R_1206_3216Metric -> Capacitor_SMD:C_1206_3216Metric
- moved R109 100.3 mm to (46.5, 72.0), turned to -90 degrees
- moved R110 97.8 mm to (48.0, 72.0), turned to -90 degrees
- moved R111 95.4 mm to (49.5, 72.0), turned to -90 degrees
- moved R112 93.0 mm to (51.0, 72.0), turned to -90 degrees
- moved R105 76.7 mm to (160.2, 61.8), turned to 90 degrees
- moved R106 75.5 mm to (161.2, 61.8), turned to 90 degrees
- moved R107 74.4 mm to (162.2, 61.8), turned to 90 degrees
- moved R108 70.6 mm to (157.5, 62.2), turned to 180 degrees
- moved R94 69.5 mm to (140.8, 61.8), turned to 90 degrees
- moved R95 68.0 mm to (141.8, 61.8), turned to 90 degrees
- moved R96 66.5 mm to (142.8, 61.8), turned to 90 degrees
- moved R97 63.4 mm to (138.0, 62.2), turned to 180 degrees
- moved R99 61.4 mm to (143.8, 61.8), turned to 90 degrees
- moved R100 60.1 mm to (144.8, 61.8), turned to 90 degrees
- moved R101 58.8 mm to (145.8, 61.8), turned to 90 degrees
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Connections:
- C10 pad 2: +5V -> +3V3
- C11 pad 2: +5V -> +3V3
- C12 pad 2: +5V -> +3V3
- C13 pad 2: +5V -> +3V3
- C14 pad 2: +5V -> +3V3
- C15 pad 2: +5V -> +3V3
- C16 pad 2: +5V -> +3V3
- C17 pad 2: +5V -> +3V3
- C19 pad 1: Net-(C19-Pad1) -> GND
- C19 pad 2: Net-(C19-Pad2) -> GND
- C20 pad 1: Net-(C20-Pad1) -> GND
- C20 pad 2: Net-(C20-Pad2) -> GND
- C21 pad 1: Net-(C19-Pad1) -> GND
- C21 pad 2: Net-(C19-Pad2) -> GND
- C22 pad 1: Net-(C20-Pad1) -> GND
- C22 pad 2: Net-(C20-Pad2) -> GND
- C23 pad 1: Net-(C23-Pad1) -> GND
- C23 pad 2: Net-(C23-Pad2) -> GND
- C24 pad 1: Net-(C23-Pad1) -> GND
- C24 pad 2: Net-(C23-Pad2) -> GND
- C25 pad 1: Net-(C25-Pad1) -> GND
- C25 pad 2: Net-(C25-Pad2) -> GND
- C26 pad 1: Net-(C25-Pad1) -> GND
- C26 pad 2: Net-(C25-Pad2) -> GND
- C27 pad 1: Net-(C27-Pad1) -> GND
- C27 pad 2: Net-(C27-Pad2) -> GND
- C28 pad 1: Net-(C27-Pad1) -> GND
- C28 pad 2: Net-(C27-Pad2) -> GND
- C29 pad 1: Net-(C29-Pad1) -> GND
- C29 pad 2: Net-(C29-Pad2) -> GND
- C30 pad 1: Net-(C29-Pad1) -> GND
- C30 pad 2: Net-(C29-Pad2) -> GND
- C33 pad 2: +5V -> Net-(SW1-A)
- C37 pad 2: +5V -> Net-(SW1-A)
- C38 pad 2: +5V -> Net-(SW1-A)
- C9 pad 2: +5V -> +3V3
- R109 pad 1: unconnected-(R109-Pad1) -> /Data
- R110 pad 1: Net-(R110-Pad1) -> /Clock
- R111 pad 1: Net-(R111-Pad1) -> /Latch
- R112 pad 1: Net-(R112-Pad1) -> /~{Clear}
- R113 pad 1: Net-(R110-Pad1) -> /Clock
- R114 pad 1: Net-(R111-Pad1) -> /Latch
- R115 pad 1: Net-(R112-Pad1) -> /~{Clear}
- R116 pad 1: Net-(R110-Pad1) -> /Clock
- R117 pad 1: Net-(R111-Pad1) -> /Latch
- R118 pad 1: Net-(R112-Pad1) -> /~{Clear}
- R119 pad 1: Net-(R110-Pad1) -> /Clock
- R120 pad 1: Net-(R111-Pad1) -> /Latch
- R121 pad 1: Net-(R112-Pad1) -> /~{Clear}
- R122 pad 1: Net-(R110-Pad1) -> /Clock
- R123 pad 1: Net-(R111-Pad1) -> /Latch
- R124 pad 1: Net-(R112-Pad1) -> /~{Clear}
- R125 pad 1: Net-(R110-Pad1) -> /Clock
- R126 pad 1: Net-(R111-Pad1) -> /Latch
- R127 pad 1: Net-(R112-Pad1) -> /~{Clear}
- R128 pad 1: Net-(R110-Pad1) -> /Clock
- R129 pad 1: Net-(R111-Pad1) -> /Latch
- R130 pad 1: Net-(R112-Pad1) -> /~{Clear}
- R131 pad 1: Net-(R110-Pad1) -> /Clock
- R132 pad 1: Net-(R111-Pad1) -> /Latch
- R133 pad 1: Net-(R112-Pad1) -> /~{Clear}
- R134 pad 1: Net-(R110-Pad1) -> /Clock
- R135 pad 1: Net-(R111-Pad1) -> /Latch
- R136 pad 1: Net-(R112-Pad1) -> /~{Clear}
- U1 pad 16: +5V -> +3V3
- U10 pad 20: unconnected-(U10-3-Pad20) -> /~{Clear}
- U10 pad 21: unconnected-(U10-2-Pad21) -> /Latch
- U10 pad 22: unconnected-(U10-1-Pad22) -> /Clock
- U10 pad 23: unconnected-(U10-0-Pad23) -> /Data
- U10 pad 3: unconnected-(U10-+3V3-Pad3) -> +3V3
- U13 pad 5: Net-(U13-KEY) -> unconnected-(U13-KEY-Pad5)
- U13 pad 8: +5V -> Net-(SW1-A)
- U2 pad 16: +5V -> +3V3
- U3 pad 16: +5V -> +3V3
- U4 pad 16: +5V -> +3V3
- U5 pad 16: +5V -> +3V3
- U6 pad 16: +5V -> +3V3
- U7 pad 16: +5V -> +3V3
- U8 pad 16: +5V -> +3V3
- U9 pad 16: +5V -> +3V3
Routing:
- net /Clock: track 0.00 -> 163.2 mm, vias 0 -> 2
- net /Latch: track 0.00 -> 161.9 mm, vias 0 -> 2
- net /~{Clear}: track 0.00 -> 161.3 mm, vias 0 -> 1
- net Net-(SW1-A): track 0.00 -> 62.3 mm, vias 0 -> 1
- net /Data: track 0.00 -> 45.0 mm, vias 0 -> 1
- net Net-(U6-Q4): track 0.49 -> 40.6 mm, vias 1 -> 2
- net GND: track 188.2 -> 228.1 mm, vias 41 -> 50
- net +3V3: track 0.00 -> 34.2 mm, vias 0 -> 6
- net Net-(Q50-B): track 0.00 -> 24.4 mm, vias 0 -> 2
- net Net-(Q51-B): track 0.00 -> 22.4 mm, vias 0 -> 2
- net Net-(Q52-B): track 0.00 -> 15.0 mm, vias 0 -> 2
- net Net-(U6-Q7): track 0.00 -> 14.3 mm, vias 0 -> 2
- net +5V: track 68.4 -> 79.4 mm, vias 6 -> 1
- net Net-(U1-DS): track 0.00 -> 9.92 mm, vias 0 -> 2
- net Net-(U1-MR#): track 0.00 -> 9.82 mm, vias 0 -> 2
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Other:
- board text added: "5V 1A"
- board text added: "Turn display OFF while programming!"
- board text added: "USB or DC jack only! DO NOT use both at once"
