File: FeriNixie ZM1177 Clock.kicad_pcb (KiCad board)
At the start: 4 copper layers, 153.5 x 98.5 mm, 323 parts, among them Q1 C20069138, Q10 C20069138, Q11 C20069138, Q12 C20069138, Q13 C20069138, Q14 C20069138, Q15 C20069138, Q16 C20069138, Q17 C20069138, Q18 C20069138, Q19 C20069138, Q2 C20069138, Q20 C20069138, Q21 C20069138, Q22 C20069138, Q23 C20069138, Q24 C20069138, Q25 C20069138, Q26 C20069138, Q27 C20069138, Q28 C20069138, Q29 C20069138, Q3 C20069138, Q30 C20069138, Q31 C20069138, Q32 C20069138, Q33 C20069138, Q34 C20069138, Q35 C20069138, Q36 C20069138, Q37 C20069138, Q38 C20069138, Q39 C20069138, Q4 C20069138, Q40 C20069138, Q41 C20069138, Q42 C20069138, Q43 C20069138, Q44 C20069138, Q45 C20069138, Q46 C20069138, Q47 C20069138, Q48 C20069138, Q49 C20069138, Q5 C20069138, Q50 C20069138, Q51 C20069138, Q52 C20069138, Q53 C20069138, Q54 C20069138, Q55 C20069138, Q56 C20069138, Q57 C20069138, Q58 C20069138, Q59 C20069138, Q6 C20069138, Q60 C20069138, Q61 C20069138, Q62 C20069138, Q63 C20069138, Q64 C20069138, Q65 C20069138, Q66 C20069138, Q67 C20069138, Q68 C20069138, Q69 C20069138, Q7 C20069138, Q70 C20069138, Q71 C20069138, Q72 C20069138, Q8 C20069138, Q9 C20069138, U1 74HC595D,118, U10 RP2040-Tiny, U11 NCH8200HV, U12 1SMA4740A_C19077479, U13 IP5306, U14 TYPE-C_16PIN_2MD(073), U15 KT-0603R, U16 KT-0603R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

Commit message: Push all changes
Parts:
- removed R257, R258, R259, R260, R261: 5.1K, Resistor_SMD:R_0402_1005Metric
- added G***: LOGO, NixMotes:nix_big_sexy_headbust_18mm, B.Cu at (140.0, 99.5)
- added R150: 100K, Resistor_SMD:R_1206_3216Metric, F.Cu at (56.5, 110.5)
- added R151: 100K, Resistor_SMD:R_1206_3216Metric, F.Cu at (54.0, 113.0)
Routing:
- net USB5V: track 92.5 -> 89.3 mm, vias 4 -> 3
- net GND: track 1322.0 -> 1324.6 mm
- net Net-(U10-29): track 8.83 -> 10.5 mm
- net Net-(R258-Pad2): track 1.03 -> 0.00 mm
- net Net-(R260-Pad2): track 1.00 -> 0.00 mm
- net Net-(R259-Pad2): track 1.00 -> 0.00 mm
Other:
- board text added: "FeriNixie ZM1177 Clock V1 by Ferinix NCH8200HV Boost 5V 3A USB C in 18650 Battery Backup + Charger"
- board text removed: "ZM1177 Clock V1 NCH8200HV Boost 5V 1A USB C in"
