File: FeriNixie ZM1177 Clock.kicad_sch (KiCad schematic)
At the start: 254 parts, among them Q1 C20069138, Q10 C20069138, Q11 C20069138, Q12 C20069138, Q13 C20069138, Q14 C20069138, Q15 C20069138, Q16 C20069138, Q17 C20069138, Q18 C20069138, Q19 C20069138, Q2 C20069138, Q20 C20069138, Q21 C20069138, Q22 C20069138, Q23 C20069138, Q24 C20069138, Q25 C20069138, Q26 C20069138, Q27 C20069138, Q28 C20069138, Q29 C20069138, Q3 C20069138, Q30 C20069138, Q31 C20069138, Q32 C20069138, Q33 C20069138, Q34 C20069138, Q35 C20069138, Q36 C20069138, Q37 C20069138, Q38 C20069138, Q39 C20069138, Q4 C20069138, Q40 C20069138, Q41 C20069138, Q42 C20069138, Q43 C20069138, Q44 C20069138, Q45 C20069138, Q46 C20069138, Q47 C20069138, Q48 C20069138, Q49 C20069138, Q5 C20069138, Q50 C20069138, Q51 C20069138, Q52 C20069138, Q53 C20069138, Q54 C20069138, Q55 C20069138, Q56 C20069138, Q57 C20069138, Q58 C20069138, Q59 C20069138, Q6 C20069138, Q60 C20069138, Q61 C20069138, Q62 C20069138, Q63 C20069138, Q64 C20069138, Q65 C20069138, Q66 C20069138, Q67 C20069138, Q68 C20069138, Q69 C20069138, Q7 C20069138, Q70 C20069138, Q8 C20069138, Q9 C20069138, U1 74HC595D,118, U2 74HC595D,118, U3 74HC595D,118, U4 74HC595D,118, U5 74HC595D,118, U6 74HC595D,118, U7 74HC595D,118, U8 74HC595D,118, U9 74HC595D,118

Commit message: Significant upgrades
Parts:
- added C18, C31: 10uF, Capacitor_SMD:C_0402_1005Metric, symbol NixMinis:Mini_C
- added U10: RP2040-Tiny, NixFootprints:RP2040-Tiny Package, symbol NixSymbols:RP2040-Tiny-Waveshare
- added U11: NCH8200HV, NixFootprints:NCH8200HV Through-Hole, symbol NixSymbols:NCH8200HV
- added U12: 1SMA4740A_C19077479, footprint:SMA_L4.3-W2.6-LS5.0-RD, symbol JLCPCB_Imported:1SMA4740A_C19077479
Connections:
- net +170V: now also C31.2, U11.2 (170V)
- net +5V: now also C18.2, U10.1 (+5V), U11.1 (12V), U12.1 (K)
- net GND: now also C18.1, C31.1, U10.2 (GND), U11.3 (GND), U11.4 (GND), U12.2 (A)
- net at R21.1: now also U9.2 (Q2)
- net at U9.3 (Q3): now also R22.1
- net at U9.4 (Q4): now also R23.1
- net at U9.5 (Q5): now also R24.1

Commit message: publish updates
Parts:
- removed C18, C31: 10uF, Capacitor_SMD:C_0402_1005Metric, symbol NixMinis:Mini_C
- added BT1: Battery_Cell, Battery:BatteryHolder_Keystone_1042_1x18650, symbol Device:Battery_Cell
- added C18: C, Capacitor_THT:C_Radial_D8.0mm_H11.5mm_P3.50mm, symbol Device:C_Polarized
- added C32, C33, C37, C38: CL31A226KAHNNNE, Capacitor_SMD:C_1206_3216Metric, symbol JLCPCB_Imported:CL31A226KAHNNNE
- added C34, C35, C36, C39: CL10A106KP8NNNC, Capacitor_SMD:C_0603_1608Metric, symbol JLCPCB_Imported:CL10A106KP8NNNC
- added L1: FTM201610C1R0MCTA, JLCPCB_Imported:L0806, symbol JLCPCB_Imported:FTM201610C1R0MCTA
- added R137: R, Resistor_THT:R_Axial_DIN0414_L11.9mm_D4.5mm_P15.24mm_Horizontal, symbol Device:R
- added R138, R139: 0603WAF200KT5E, Resistor_SMD:R_0603_1608Metric, symbol JLCPCB_Imported:0603WAF200KT5E
- added R254, R255: 5.1K, Resistor_SMD:R_0402_1005Metric, symbol NixMinis:Mini_R
- added R256: 10K, Resistor_SMD:R_0402_1005Metric, symbol NixMinis:Mini_R
- added U13: IP5306, JLCPCB_Imported:ESOP-8_L4.9-W3.9-P1.27-LS6.0-BL-EP, symbol JLCPCB_Imported:IP5306
- added U14: TYPE-C_16PIN_2MD(073), JLCPCB_Imported:USB-C-SMD_TYPE-C-16PIN-2MD-073, symbol JLCPCB_Imported:TYPE-C_16PIN_2MD(073)
- added U15, U16, U17, U18: KT-0603R, JLCPCB_Imported:LED-SMD_L1.6-W0.8-R-RD, symbol JLCPCB_Imported:KT-0603R
- added U19: TS-1187A-B-A-B, JLCPCB_Imported:SW-SMD_4P-L5.1-W5.1-P3.70-LS6.5-TL_H1.5, symbol JLCPCB_Imported:TS-1187A-B-A-B
- C1, C2, C3, C4, C5, C6: footprint Capacitor_SMD:C_1206_3216Metric -> Resistor_SMD:R_1206_3216Metric
- C19, C20, C21, C22, C23, C24, C25, C26, C27, C28, C29, C30: footprint Capacitor_SMD:C_1206_3216Metric -> (none)
- R11: now in the parts list
- U10: footprint NixFootprints:RP2040-Tiny Package -> NixFootprints:RP2040-Tiny Package Extra Clearance; now left out of the parts list
- U11: now left out of the parts list
- U12: footprint footprint:SMA_L4.3-W2.6-LS5.0-RD -> JLCPCB_Imported:SMA_L4.3-W2.6-LS5.0-RD
Connections:
- net +170V: now also C18.1
- net +5V: now also C33.2, C37.2, C38.2, C39.2, U13.8 (VOUT)
- net GND: now also BT1.2 (-), C18.2, C32.1, C33.1, C34.1, C35.1, C36.1, C37.1, C38.1, C39.1, R254.1, R255.1, U13.9 (EP), U14.13 (EH), U14.14 (EH), U14.A1B12 (GND), U14.B1A12 (GND), U19.1 (A)
- new net: U13.3 (LED2), U17.1 (A), U18.2 (K)
- new net: U13.4 (LED3), U15.2 (K), U16.1 (A), U17.2 (K), U18.1 (A)
- new net: U13.2 (LED1), U15.1 (A), U16.2 (K)
- new net: C35.2, R137.2, R139.2, U13.1 (VIN)
- new net: R255.2, U14.A5 (CC1)
- new net: U14.A6 (Dp1), U14.B7 (Dn2)
- new net: U14.A7 (Dn1), U14.B6 (Dp2)
- new net: R254.2, U14.B5 (CC2)
- new net: R256.1, U13.5 (KEY)
- new net: R256.2, U19.2 (B)
- new net: L1.1, U13.7 (SW)
- new net: C34.2, R139.1
- new net: C36.2, R138.1
- new net USB5V: R137.1, U14.A4B9 (VBUS), U14.B4A9 (VBUS)
- new net VBAT: BT1.1 (+), C32.2, L1.2, R138.2, U13.6 (BAT)
- no-connect marks 1 -> 4

Commit message: PCB updates
Parts:
- removed R256: 10K, Resistor_SMD:R_0402_1005Metric, symbol NixMinis:Mini_R
- removed U19: TS-1187A-B-A-B, JLCPCB_Imported:SW-SMD_4P-L5.1-W5.1-P3.70-LS6.5-TL_H1.5, symbol JLCPCB_Imported:TS-1187A-B-A-B
Connections:
- no-connect marks 4 -> 5
Changed lines of the file:
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@@
 	)
 	(junction
-		(at 106.68 179.07)
-		(diameter 0)
-		(color 0 0 0 0)
-	)
-	(junction
 		(at 106.68 59.69)
 		(diameter 0)
@@
 		(at 15.24 48.26)
 	)
+	(no_connect
+		(at 106.68 163.83)
+	)
 	(wire
 		(pts
@@
 	(wire
 		(pts
-			(xy 74.93 179.07) (xy 106.68 179.07)
+			(xy 74.93 179.07) (xy 123.19 179.07)
 		)
 		(stroke
@@
 	(wire
 		(pts
-			(xy 106.68 179.07) (xy 123.19 179.07)
-		)
-		(stroke
-			(width 0)
-			(type default)
-		)
-	)
-	(wire
-		(pts
 			(xy 73.66 64.77) (xy 76.2 64.77)
 		)
@@
 	(wire
 		(pts
-			(xy 106.68 179.07) (xy 106.68 177.8)
-		)
-		(stroke
-			(width 0)
-			(type default)
-		)
-	)
-	(wire
-		(pts
 			(xy 137.16 64.77) (xy 139.7 64.77)
 		)
@@
 	(symbol
 		(lib_id "NixMinis:Mini_R")
-		(at 106.68 167.64 90)
-		(mirror x)
-		(unit 1)
-		(body_style 1)
-		(exclude_from_sim no)
-		(in_bom yes)
-		(on_board yes)
-		(in_pos_files yes)
-		(dnp no)
-		(fields_autoplaced yes)
-		(property "Reference" "R256"
-			(at 105.9096 165.7187 0)
-			(hide yes)
-			(show_name no)
-			(do_not_autoplace yes)
-			(effects
-				(font
-					(size 0.635 0.635)
-				)
-				(justify bottom)
-			)
-		)
-		(property "Value" "10K"
-			(at 106.676 165.7454 0)
-			(show_name no)
-			(do_not_autoplace yes)
-			(effects
-				(font
-					(size 0.381 0.381)
-				)
-			)
-		)
-		(property "Footprint" "Resistor_SMD:R_0402_1005Metric"
-			(at 106.68 167.64 0)
-			(hide yes)
-			(show_name no)
-			(do_not_autoplace no)
-			(effects
-				(font
-					(size 1.27 1.27)
-				)
-			)
-		)
-		(property "Datasheet" ""
-			(at 101.092 168.91 90)
-			(hide yes)
-			(show_name no)
-			(do_not_autoplace yes)
-			(effects
-				(font
-					(size 0.635 0.635)
-				)
-			)
-		)
-		(property "Description" "Resistor, small symbol"
-			(at 98.552 167.64 0)
-			(hide yes)
-			(show_name no)
-			(do_not_autoplace no)
-			(effects
-				(font
-					(size 1.27 1.27)
-				)
-			)
-		)
-		(pin "2"
-		)
-		(pin "1"
-		)
-		(instances
-			(project "FeriNixie ZM1177 Clock"
-				(path "/c395a452-49ff-4706-a1e4-e3a262b74a6a"
-					(reference "R256")
-					(unit 1)
-				)
-			)
-		)
-	)
-	(symbol
-		(lib_id "NixMinis:Mini_R")
 		(at 187.96 63.5 90)
 		(unit 1)
@@
 					(unit 1)
 				)
-			)
-		)
-	)
-	(symbol
-		(lib_id "JLCPCB_Imported:TS-1187A-B-A-B")
-		(at 109.22 172.72 90)
-		(unit 1)
-		(body_style 1)
-		(exclude_from_sim no)
-		(in_bom yes)
-		(on_board yes)
-		(in_pos_files yes)
-		(dnp no)
-		(fields_autoplaced yes)
-		(property "Reference" "U19"
-			(at 115.57 171.4499 90)
-			(show_name no)
-			(do_not_autoplace no)
-			(effects
-				(font
-					(size 1.27 1.27)
-				)
-				(justify right)
-			)
-		)
-		(property "Value" "TS-1187A-B-A-B"
-			(at 115.57 173.9899 90)
-			(show_name no)
-			(do_not_autoplace no)
-			(effects
-				(font
-					(size 1.27 1.27)
-				)
-				(justify right)
-			)
-		)
-		(property "Footprint" "JLCPCB_Imported:SW-SMD_4P-L5.1-W5.1-P3.70-LS6.5-TL_H1.5"
-			(at 119.38 172.72 0)
-			(hide yes)
-			(show_name no)
-			(do_not_autoplace no)
-			(effects
-				(font
-					(size 1.27 1.27)
-					(italic yes)
-				)
-			)
-		)
-		(property "Datasheet" "https://item.szlcsc.com/datasheet/TS-1187A-C-6.0-B/299982.html"
-			(at 109.093 175.006 0)
-			(hide yes)
-			(show_name no)
-			(do_not_autoplace no)
-			(effects
-				(font
-					(size 1.27 1.27)
-				)
-				(justify left)
-			)
-		)
-		(property "Description" ""
-			(at 109.22 172.72 0)
-			(hide yes)
-			(show_name no)
-			(do_not_autoplace no)
-			(effects
-				(font
-					(size 1.27 1.27)
-				)
-			)
-		)
-		(property "LCSC" "C318884"
-			(at 109.22 172.72 0)
-			(hide yes)
-			(show_name no)
-			(do_not_autoplace no)
-			(effects
-				(font
-					(size 1.27 1.27)
-				)
-			)
-		)
-		(pin "2"
-		)
-		(pin "1"
-		)
-		(pin "4"
-		)
-		(pin "3"
-		)
-		(instances
-			(project "FeriNixie ZM1177 Clock"
-				(path "/c395a452-49ff-4706-a1e4-e3a262b74a6a"
-					(reference "U19")
-					(unit 1)
-				)

Commit message: Lots of improvements and adjustments
Parts:
- added R140: 100K, Resistor_SMD:R_1206_3216Metric, symbol NixMinis:Mini_R
- added SW1: SW_SPST, NixFootprints:SW_SPST_R1966ABLKBLKFR, symbol Switch:SW_SPST
- C1, C2, C3, C4, C5, C6: footprint Resistor_SMD:R_1206_3216Metric -> Capacitor_SMD:C_1206_3216Metric
Connections:
- net +5V: now also SW1.2 (B); no longer C10.2, C11.2, C12.2, C13.2, C14.2, C15.2, C16.2, C17.2, C33.2, C37.2, C38.2, C9.2, U1.16 (VCC), U13.8 (VOUT), U2.16 (VCC), U3.16 (VCC), U4.16 (VCC), U5.16 (VCC), U6.16 (VCC), U7.16 (VCC), U8.16 (VCC), U9.16 (VCC)
- net GND: now also C19.1, C19.2, C20.1, C20.2, C21.1, C21.2, C22.1, C22.2, C23.1, C23.2, C24.1, C24.2, C25.1, C25.2, C26.1, C26.2, C27.1, C27.2, C28.1, C28.2, C29.1, C29.2, C30.1, C30.2, R140.2
- net Clock: now reaches R110.1, R113.1, R116.1, R119.1, R122.1, R125.1, R128.1, R131.1, R134.1
- net Clock: now also U10.22 (1)
- net Latch: now reaches R111.1, R114.1, R117.1, R120.1, R123.1, R126.1, R129.1, R132.1, R135.1
- net Latch: now also U10.21 (2)
- net ~{Clear}: now reaches U10.20 (3)
- net ~{Clear}: now also R112.1, R115.1, R118.1, R121.1, R124.1, R127.1, R130.1, R133.1, R136.1
- net Data: now reaches U10.23 (0)
- net Data: now also R109.1
- net +3V3: now reaches U10.3 (+3V3)
- net +3V3: now also C10.2, C11.2, C12.2, C13.2, C14.2, C15.2, C16.2, C17.2, C9.2, U1.16 (VCC), U2.16 (VCC), U3.16 (VCC), U4.16 (VCC), U5.16 (VCC), U6.16 (VCC), U7.16 (VCC), U8.16 (VCC), U9.16 (VCC)
- new net: C33.2, C37.2, C38.2, R140.1, SW1.1 (A), U13.8 (VOUT)
