File: FeriNixie ZM1177 Clock.kicad_sch (KiCad schematic)
At the start: 281 parts, among them Q1 C20069138, Q10 C20069138, Q11 C20069138, Q12 C20069138, Q13 C20069138, Q14 C20069138, Q15 C20069138, Q16 C20069138, Q17 C20069138, Q18 C20069138, Q19 C20069138, Q2 C20069138, Q20 C20069138, Q21 C20069138, Q22 C20069138, Q23 C20069138, Q24 C20069138, Q25 C20069138, Q26 C20069138, Q27 C20069138, Q28 C20069138, Q29 C20069138, Q3 C20069138, Q30 C20069138, Q31 C20069138, Q32 C20069138, Q33 C20069138, Q34 C20069138, Q35 C20069138, Q36 C20069138, Q37 C20069138, Q38 C20069138, Q39 C20069138, Q4 C20069138, Q40 C20069138, Q41 C20069138, Q42 C20069138, Q43 C20069138, Q44 C20069138, Q45 C20069138, Q46 C20069138, Q47 C20069138, Q48 C20069138, Q49 C20069138, Q5 C20069138, Q50 C20069138, Q51 C20069138, Q52 C20069138, Q53 C20069138, Q54 C20069138, Q55 C20069138, Q56 C20069138, Q57 C20069138, Q58 C20069138, Q59 C20069138, Q6 C20069138, Q60 C20069138, Q61 C20069138, Q62 C20069138, Q63 C20069138, Q64 C20069138, Q65 C20069138, Q66 C20069138, Q67 C20069138, Q68 C20069138, Q69 C20069138, Q7 C20069138, Q70 C20069138, Q8 C20069138, Q9 C20069138, SW1 SW_SPST, U1 74HC595D,118, U10 RP2040-Tiny, U11 NCH8200HV, U12 1SMA4740A_C19077479, U13 IP5306, U14 TYPE-C_16PIN_2MD(073), U15 KT-0603R, U16 KT-0603R, U17 KT-0603R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

Commit message: Push changes
Parts:
- removed R137: R, Resistor_THT:R_Axial_DIN0414_L11.9mm_D4.5mm_P15.24mm_Horizontal, symbol Device:R
- added C31, C40, C41, C42: 1uF, Resistor_SMD:R_0402_1005Metric, symbol NixMinis:Mini_C
- added C43: 100nF, Capacitor_SMD:C_1206_3216Metric, symbol NixMinis:Mini_C
- added NE5, NE6: (no value), FeriNixie:NeonIndicator_2ML_1MH_B10A, symbol FeriNixie:NeonIndicator_2ML_1MH_B10A
- added Q71, Q72: C20069138, JLCPCB_Imported:SOT-23-3_L2.9-W1.3-P1.90-LS2.4-BR, symbol NixMinis:Mini_BJT_NPN
- added R137, R147: 10K, Resistor_SMD:R_0402_1005Metric, symbol NixMinis:Mini_R
- added R141, R142, R143, R144: 1K, Capacitor_SMD:C_0402_1005Metric, symbol NixMinis:Mini_R
- added R145, R146, R148, R149: 100K, Resistor_SMD:R_1206_3216Metric, symbol NixMinis:Mini_R
- added R257, R258, R259, R260, R261: 5.1K, Resistor_SMD:R_0402_1005Metric, symbol NixMinis:Mini_R
- added U19, U20, U21, U22: TS-1187A-B-A-B, JLCPCB_Imported:SW-SMD_4P-L5.1-W5.1-P3.70-LS6.5-TL_H1.5, symbol JLCPCB_Imported:TS-1187A-B-A-B
- SW1: footprint NixFootprints:SW_SPST_R1966ABLKBLKFR -> NixFootprints:SW_SPST_L101011MS02Q
Connections:
- net +170V: now also C43.2, R145.2, R146.2, R148.2, R149.2
- net GND: now also C31.1, C40.1, C41.1, C42.1, C43.1, Q71.2 (E), Q72.2 (E), R257.1, U19.3 (C), U19.4 (D), U20.3 (C), U20.4 (D), U21.3 (C), U21.4 (D), U22.3 (C), U22.4 (D)
- net USB5V: now also C35.2, R139.2, U13.1 (VIN), R261.2
- net IN_Adjust: now reaches U10.16 (7)
- net IN_Adjust: now also R144.1
- net IN_Select: now reaches U10.17 (6)
- net IN_Select: now also R143.1
- net IN_Light: now reaches U10.18 (5)
- net IN_Light: now also R142.1
- net IN_Toggle: now reaches U10.19 (4)
- net IN_Toggle: now also R141.1
- net at U10.4 (29): now also R257.2, R258.1
- net at U9.6 (Q6): now also R137.1
- net at U9.7 (Q7): now also R147.1
- new net: NE5.2 (K), NE6.1 (A), Q71.3 (C), R145.1, R146.1
- new net: R258.2, R259.1
- new net: C41.2, R143.2, U21.1 (A), U21.2 (B)
- new net: C40.2, R142.2, U20.1 (A), U20.2 (B)
- new net: NE5.1 (A), NE6.2 (K), Q72.3 (C), R148.1, R149.1
- new net: Q72.1 (B), R147.2
- new net: C42.2, R144.2, U22.1 (A), U22.2 (B)
- new net: Q71.1 (B), R137.2
- new net: R259.2, R260.1
- new net: R260.2, R261.1
- new net: C31.2, R141.2, U19.1 (A), U19.2 (B)

Commit message: Push all changes
Parts:
- removed R257, R258, R259, R260, R261: 5.1K, Resistor_SMD:R_0402_1005Metric, symbol NixMinis:Mini_R
- added R150, R151: 100K, Resistor_SMD:R_1206_3216Metric, symbol NixMinis:Mini_R
Connections:
- net GND: now also R151.2
- net USB5V: now also R150.1
- net at U10.4 (29): now also R150.2, R151.1
