File: FeriNixie ZM1177 Clock_Bottom.kicad_pcb (KiCad board)
At the start: 2 copper layers, 153.5 x 49 mm, 51 parts, among them U10 RP2040-Tiny, U11 NCH8200HV, U12 1SMA4740A_C19077479, U13 IP5306, U14 TYPE-C_16PIN_2MD(073), U15 KT-0603R, U16 KT-0603R, U17 KT-0603R, U18 KT-0603R, U19 TS-1187A-B-A-B, U20 TS-1187A-B-A-B, U21 TS-1187A-B-A-B, U22 TS-1187A-B-A-B

Commit message: Push all changes
Parts:
- removed R257, R258, R259, R260, R261: 5.1K, Resistor_SMD:R_0402_1005Metric
- added G***: LOGO, NixMotes:nix_big_sexy_headbust_18mm, B.Cu at (140.0, 50.0)
- added R150: 100K, Resistor_SMD:R_1206_3216Metric, F.Cu at (56.5, 61.0)
- added R151: 100K, Resistor_SMD:R_1206_3216Metric, F.Cu at (54.0, 63.5)
Routing:
- net USB5V: track 92.5 -> 89.3 mm, vias 4 -> 3
- net GND: track 281.0 -> 283.6 mm
- net Net-(U10-29): track 8.83 -> 10.5 mm
- net Net-(R258-Pad2): track 1.03 -> 0.00 mm
- net Net-(R260-Pad2): track 1.00 -> 0.00 mm
- net Net-(R259-Pad2): track 1.00 -> 0.00 mm
Other:
- copper layers 2 -> 4
- board text added: "FeriNixie ZM1177 Clock V1 by Ferinix NCH8200HV Boost 5V 3A USB C in 18650 Battery Backup + Charger"
- board text removed: "ZM1177 Clock V1 NCH8200HV Boost 5V 1A USB C in"
