File: FeriNixie ZM1177 Clock_Top.kicad_pcb (KiCad board)
At the start: 4 copper layers, 153.5 x 98.5 mm, 323 parts, among them Q1 C20069138, Q10 C20069138, Q11 C20069138, Q12 C20069138, Q13 C20069138, Q14 C20069138, Q15 C20069138, Q16 C20069138, Q17 C20069138, Q18 C20069138, Q19 C20069138, Q2 C20069138, Q20 C20069138, Q21 C20069138, Q22 C20069138, Q23 C20069138, Q24 C20069138, Q25 C20069138, Q26 C20069138, Q27 C20069138, Q28 C20069138, Q29 C20069138, Q3 C20069138, Q30 C20069138, Q31 C20069138, Q32 C20069138, Q33 C20069138, Q34 C20069138, Q35 C20069138, Q36 C20069138, Q37 C20069138, Q38 C20069138, Q39 C20069138, Q4 C20069138, Q40 C20069138, Q41 C20069138, Q42 C20069138, Q43 C20069138, Q44 C20069138, Q45 C20069138, Q46 C20069138, Q47 C20069138, Q48 C20069138, Q49 C20069138, Q5 C20069138, Q50 C20069138, Q51 C20069138, Q52 C20069138, Q53 C20069138, Q54 C20069138, Q55 C20069138, Q56 C20069138, Q57 C20069138, Q58 C20069138, Q59 C20069138, Q6 C20069138, Q60 C20069138, Q61 C20069138, Q62 C20069138, Q63 C20069138, Q64 C20069138, Q65 C20069138, Q66 C20069138, Q67 C20069138, Q68 C20069138, Q69 C20069138, Q7 C20069138, Q70 C20069138, Q71 C20069138, Q72 C20069138, Q8 C20069138, Q9 C20069138, U1 74HC595D,118, U10 RP2040-Tiny, U11 NCH8200HV, U12 1SMA4740A_C19077479, U13 IP5306, U14 TYPE-C_16PIN_2MD(073), U15 KT-0603R, U16 KT-0603R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

Commit message: Push all changes
Parts:
- removed the ? at (45.2, 80.2)
- removed the ? at (45.2, 83.2)
- removed BT1: Battery_Cell, Battery:BatteryHolder_Keystone_1042_1x18650
- removed C18: C, Capacitor_THT:C_Radial_D8.0mm_H11.5mm_P3.50mm
- removed C31, C40, C41, C42: 1uF, Resistor_SMD:R_0402_1005Metric
- removed C32, C33, C37, C38: CL31A226KAHNNNE, Capacitor_SMD:C_1206_3216Metric
- removed C34, C35, C36, C39: CL10A106KP8NNNC, Capacitor_SMD:C_0603_1608Metric
- removed L1: FTM201610C1R0MCTA, JLCPCB_Imported:L0806
- removed R138, R139: 0603WAF200KT5E, Resistor_SMD:R_0603_1608Metric
- removed R140: 100K, Resistor_SMD:R_1206_3216Metric
- removed R141, R142, R143, R144: 1K, Capacitor_SMD:C_0402_1005Metric
- removed R254, R255, R257, R258, R259, R260, R261: 5.1K, Resistor_SMD:R_0402_1005Metric
- removed the REF** at (102.2, 80.0)
- removed the REF** at (49.5, 117.0)
- removed the REF** at (174.0, 99.5)
- removed the REF** at (154.5, 78.0)
- removed the REF** at (30.5, 99.5)
- removed the REF** at (50.0, 78.0)
- removed SW: L101011MS02Q, NixFootprints:SW_SPST_L101011MS02Q
- removed U10: RP2040-Tiny, NixFootprints:RP2040-Tiny Package Extra Clearance
- removed U11: NCH8200HV, NixFootprints:NCH8200HV Through-Hole
- removed U12: 1SMA4740A_C19077479, JLCPCB_Imported:SMA_L4.3-W2.6-LS5.0-RD
- removed U13: IP5306, JLCPCB_Imported:ESOP-8_L4.9-W3.9-P1.27-LS6.0-BL-EP
- removed U14: TYPE-C_16PIN_2MD(073), JLCPCB_Imported:USB-C-SMD_TYPE-C-16PIN-2MD-073
- removed U15, U16, U17, U18: KT-0603R, JLCPCB_Imported:LED-SMD_L1.6-W0.8-R-RD
- removed U19, U20, U21, U22: TS-1187A-B-A-B, JLCPCB_Imported:SW-SMD_4P-L5.1-W5.1-P3.70-LS6.5-TL_H1.5
Routing:
- net GND: track 1322.0 -> 1041.0 mm, vias 85 -> 81
- net /IN_Adjust: track 113.9 -> 0.00 mm, vias 1 -> 0
- net /IN_Select: track 107.1 -> 0.00 mm, vias 1 -> 0
- net /IN_Light: track 100.2 -> 0.00 mm, vias 1 -> 0
- net /IN_Toggle: track 93.3 -> 0.00 mm, vias 1 -> 0
- net USB5V: track 92.5 -> 0.00 mm, vias 4 -> 0
- net +5V: track 85.1 -> 0.00 mm, vias 1 -> 0
- net Net-(SW1-A): track 65.1 -> 0.00 mm, vias 1 -> 0
- net /~{Clear}: track 207.7 -> 175.6 mm
- net /Latch: track 213.4 -> 183.4 mm
- net /Clock: track 220.7 -> 192.2 mm
- net /Data: track 45.0 -> 18.0 mm
- net Net-(Q28-B): track 0.00 -> 26.5 mm, vias 0 -> 2
- net VBAT: track 21.5 -> 0.00 mm
- net Net-(U13-LED3): track 16.9 -> 0.00 mm
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Other:
- board size 153.5 x 98.5 mm -> 153.5 x 49 mm
- board text removed: "18650 3.7V Lithium Ion Battery Only"
- board text removed: "25 50 75 100"
- board text removed: "Adjust"
- board text removed: "Brightness"
- board text removed: "Charge"
- board text removed: "Select"
- board text removed: "Toggle"
- board text removed: "Turn display OFF while programming!"
- board text removed: "ZM1177 Clock V1 NCH8200HV Boost 5V 1A USB C in"
